File: Hardware/MakerTherapyBadge.brd (EAGLE design)
At the start: 100 x 80 mm, 0 parts

Commit message: progress from march 6
Parts:
- added C1, C3: 0.1u, LinnesLab-Passives:C0603
- added C2: 2.2u, LinnesLab-Passives:C0603
- added C4, C5: 22p, LinnesLab-Passives:C0603
- added C6: 4.7u, LinnesLab-Passives:C0603
- added D2: (no value), LinnesLab-DiscreteSemi:USC
- added D4: 1A/23V/620mV, LinnesLab-DiscreteSemi:USC
- added FTDI1: FTDI_DEVICE, LinnesLab-Connectors:FTDI_DEVICE
- added J1: AVR_SPI_PROG_3X2NS, LinnesLab-Connectors:2X3-NS
- added LIPO1: (no value), LinnesLab-Connectors:JST-2-SMD
- added ON/OFF: SWITCH.JS202011JXQNUPWARDS, LinnesLab-Switches:SWITCH.00
- added R1: 10k, LinnesLab-Passives:R0603
- added RESET: (no value), LinnesLab-Switches:BUTTON-GULLWING
- added U1: ATMEGA328P_TQFP, LinnesLab-Microcontrollers:TQFP32-08
- added XTAL: (no value), LinnesLab-Clocks:CA-301
Connections:
- new net DTR: C1.2
- new net GND: C2.2, C3.2, C4.2, C5.2, C6.2, J1.6, LIPO1.1, RESET.3, RESET.4, U1.21, U1.3, U1.5
- new net N$1: FTDI1.DTR, FTDI1.TXO
- new net N$11: J1.1
- new net N$12: J1.3
- new net N$13: J1.5
- new net N$2: D2.+, FTDI1.RXI
- new net N$3: FTDI1.VCC
- new net N$4: FTDI1.CTS
- new net N$5: FTDI1.GND
- new net N$6: C4.1, U1.8, XTAL.1
- new net N$7: D4.+, ON/OFF.1
- new net N$9: C5.1, U1.7, XTAL.2
- new net RESET: C1.1, R1.2, RESET.1, RESET.2, U1.29
- new net VCC: C2.1, C3.1, C6.1, D2.-, D4.-, J1.2, R1.1, U1.18, U1.4, U1.6
- new net VLIPO: LIPO1.2, ON/OFF.2
