File: Hardware/MakerTherapyBadge.brd (EAGLE design)
At the start: 100 x 80 mm, 16 parts, among them J1 AVR_SPI_PROG_3X2NS, U1 ATMEGA328P_TQFP

Commit message: finished schematic
Parts:
- added ACT, EMOJI, GAME, LED6, LED7, LT, RT: (no value), LinnesLab-LED:LED-0603
- added ACTION, LEFT, RIGHT: (no value), LinnesLab-Switches:SPST.KT11P4SM34LFS
- added C10, C13, C14, C15: 4.7u, LinnesLab-Passives:C0603
- added C11, C7: (no value), LinnesLab-Passives:C0603
- added C12, C17, C8, C9: 100n, LinnesLab-Passives:C0603
- added C16: 2.2u, LinnesLab-Passives:C0603
- added C18: 1u, LinnesLab-Passives:C0603
- added D1: 1A/23V/620mV, LinnesLab-DiscreteSemi:USC
- added LED8: (no value), adafruit:SEGMENT_BL-M12A881UR
- added MODE: SWITCH.JS202011JXQNUPWARDS, LinnesLab-Switches:SWITCH.00
- added OP1: (no value), LinnesLab-AnalogIC:SOT23-5
- added R10, R2, R3, R5: 1k, LinnesLab-Passives:R0603
- added R11, R17, R4, R7, R8: 10k, LinnesLab-Passives:R0603
- added R12: 487, LinnesLab-Passives:R0603
- added R13: 12k, LinnesLab-Passives:R0603
- added R14, R15: 210k, LinnesLab-Passives:R0603
- added R16: 3.3M, LinnesLab-Passives:R0603
- added R18, R19, R20, R21, R22, R23, R24, R25: 205, LinnesLab-Passives:R0603
- added R6, R9: (no value), LinnesLab-Passives:R0603
- added U$1: ADPS9008, LinnesLab-Sensors:6-PIN.CHIPLED
- added U3: MCP73831.SOT23-5, LinnesLab-Power:SOT23-5
- added USB1: USB.MICRO.PWR-BIGGERPADS, LinnesLab-Connectors:USB-MICRO-01.BIGGERPADS.PWR
Connections:
- new net ACTION: U1.19
- new net LD1: R22.1, U1.2
- new net LD10: J1.1, LED8.10, U1.16
- new net LD11: J1.4, LED8.11, U1.15
- new net LD12: R21.1, U1.14
- new net LD13: LED8.13, U1.13
- new net LD14: R19.1, U1.12
- new net LD15: LED8.15, U1.11
- new net LD16: LED8.16, U1.10
- new net LD2: R24.1, U1.1
- new net LD3: LED8.3, U1.32
- new net LD4: LED8.4, U1.28
- new net LD5: R25.1, U1.27
- new net LD6: LED8.6, U1.26
- new net LD7: R23.1, U1.25
- new net LD8: R20.1, U1.24
- new net LD9: J1.3, R18.1, U1.17
- new net LEFT: U1.23
- new net MODE: GAME.A, MODE.2, R2.1, U1.9
- new net N$10: LT.C, R9.2
- new net N$14: GAME.C, R3.2
- new net N$15: C9.1, LEFT.3, LEFT.4, LT.A, R8.2
- new net N$16: ACT.A, ACTION.3, ACTION.4, C7.2, R4.2
- new net N$17: ACT.C, R5.2
- new net N$18: R6.2, RT.C
- new net N$19: C8.2, R7.2, RIGHT.3, RIGHT.4, RT.A
- new net N$20: D1.+, USB1.1
- new net N$21: LED6.A, R10.1
- new net N$22: LED8.5, R25.2
- new net N$23: LED7.C, R12.2
- new net N$24: R11.2, U3.5
- new net N$25: OP1.4, R16.2, R17.1
- new net N$27: C16.2, OP1.3, R14.1, R15.2
- new net N$28: C13.2, R13.2, U$1.6
- new net N$30: C13.1, C14.1, C15.1
- new net N$31: C15.2, C16.1, R17.2
- new net N$8: EMOJI.C, R2.2
- new net PULSE: OP1.1, R16.1
- new net RIGHT: U1.22
- new net RXD: FTDI1.CTS, U1.30
- new net STAT: LED6.C, U3.1
- new net TXD: FTDI1.VCC, U1.31
- net DTR: now also FTDI1.GND
- net GND: now also C10.2, C11.2, C12.1, C14.2, C17.2, C18.2, C7.1, C8.1, C9.2, FTDI1.DTR, FTDI1.TXO, MODE.1, OP1.2, R11.1, R12.1, R13.1, R15.1, R3.1, R4.1, R5.1, R6.1, R7.1, R8.1, R9.1, U$1.4, U3.2, USB1.5
- net N$1: now also LED8.9, R18.2; no longer FTDI1.DTR, FTDI1.TXO
- net N$11: now also LED8.1, R22.2; no longer J1.1
- net N$12: now also LED8.7, R23.2; no longer J1.3
- net N$13: now also LED8.2, R24.2; no longer J1.5
- net N$3: now also LED8.14, R19.2; no longer FTDI1.VCC
- net N$4: now also LED8.8, R20.2; no longer FTDI1.CTS
- net N$5: now also LED8.12, R21.2; no longer FTDI1.GND
- net RESET: now also J1.5
- net VCC: now also ACTION.1, ACTION.2, C11.1, C12.2, C17.1, C18.1, D1.-, EMOJI.A, LED7.A, LEFT.1, LEFT.2, MODE.3, OP1.5, R10.2, R14.2, RIGHT.1, RIGHT.2, U$1.1, U3.4
- net VLIPO: now also C10.1, U3.3

Commit message: partially worked on the board
Parts:
- moved R21 340.2 mm to (54.6, 57.1), turned to 180 degrees
- moved R19 330.8 mm to (47.0, 57.1), turned to 180 degrees
- moved R18 329.9 mm to (34.3, 63.5)
- moved LED8 326.7 mm to (50.8, 39.4)
- moved R25 318.5 mm to (54.6, 19.1), flipped to the bottom
- moved R24 312.5 mm to (47.0, 19.1), turned to 180 degrees
- moved R23 312.5 mm to (58.4, 19.1), turned to 180 degrees
- moved R22 303.7 mm to (41.9, 19.1), turned to 180 degrees
- moved R20 303.1 mm to (62.2, 19.1), turned to 180 degrees
- moved USB1 188.6 mm to (20.3, 48.3)
- moved LIPO1 166.4 mm to (92.7, 73.7)
- moved J1 119.7 mm to (8.89, 62.2)
- moved FTDI1 111.9 mm to (50.5, 66.0)
- moved C1 95.6 mm to (83.8, 21.6)
- moved C2 95.6 mm to (83.8, 17.8)
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
Commit message: updates from 3/20
Parts:
- C7: value (none) -> 100n
- R6, R9: value (none) -> 1k
- moved OP1 325.3 mm to (42.0, 65.9), flipped to the bottom
- moved R14 324.4 mm to (38.7, 61.7), flipped to the bottom
- moved C18 319.8 mm to (46.6, 66.2), flipped to the bottom, turned to 270 degrees
- moved C17 316.9 mm to (49.2, 66.1), flipped to the bottom, turned to 270 degrees
- moved LED7 312.0 mm to (7.59, 63.8), turned to 180 degrees
- moved C16 308.2 mm to (36.8, 64.6), flipped to the bottom
- moved C15 303.4 mm to (32.4, 64.6), flipped to the bottom, turned to 180 degrees
- moved C14 298.0 mm to (28.8, 63.7), flipped to the bottom, turned to 270 degrees
- moved R17 294.6 mm to (37.3, 69.3), flipped to the bottom
- moved C13 294.4 mm to (25.7, 64.6), flipped to the bottom, turned to 180 degrees
- moved R16 292.2 mm to (41.8, 69.3), flipped to the bottom
- moved C12 288.2 mm to (17.4, 64.0), flipped to the bottom, turned to 270 degrees
- moved R15 281.9 mm to (43.1, 61.7), flipped to the bottom
- moved R13 270.7 mm to (22.9, 63.7), flipped to the bottom, turned to 90 degrees
- moved R12 262.7 mm to (3.35, 63.8), flipped to the bottom, turned to 180 degrees
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Other:
- board size 100 x 80 mm -> 63.5 x 85.7 mm

Commit message: slight new updates 3/20
Parts:
- moved LT 3.62 mm to (15.4, 18.8)
- moved R9 3.59 mm to (15.4, 15.9)
- moved R7 3.56 mm to (48.8, 15.5), turned to 0 degrees
- moved RT 3.36 mm to (55.6, 18.3)
- moved RIGHT 3.15 mm to (52.1, 10.4)
- moved R6 3.06 mm to (55.7, 15.6)
- moved R4 2.81 mm to (28.3, 15.2)
- moved C7 2.62 mm to (28.2, 17.6)
- moved C8 2.53 mm to (48.8, 18.4), turned to 0 degrees
- moved ACT 1.69 mm to (35.6, 17.7)
- moved ACTION 1.60 mm to (31.8, 10.4)
- moved R5 1.53 mm to (35.7, 15.4)
- moved LEFT 1.30 mm to (11.4, 10.4), turned to 180 degrees
- moved C9 0.40 mm to (7.06, 18.7)
Routing:
- net N$19: track 0.00 -> 24.1 mm
- net N$15: track 0.00 -> 21.5 mm
- net N$16: track 0.00 -> 20.4 mm
- net N$10: track 0.00 -> 3.03 mm
- net N$18: track 0.00 -> 2.82 mm
- net N$17: track 0.00 -> 2.56 mm

Commit message: changes after 3/27
Parts:
- moved LED7 52.0 mm to (58.3, 52.4)
- moved R12 49.5 mm to (51.6, 52.4)
- moved FTDI1 35.4 mm to (31.4, 22.5), flipped to the bottom, turned to 0 degrees
- moved D2 34.2 mm to (31.5, 20.2), turned to 0 degrees
- moved RESET 22.0 mm to (11.8, 30.4)
- moved C1 21.7 mm to (12.9, 25.5)
- moved R1 21.5 mm to (12.9, 27.4)
- moved J1 16.1 mm to (10.5, 60.4), turned to 0 degrees
- moved EMOJI 15.0 mm to (4.19, 44.6), turned to 270 degrees
- moved C4 14.8 mm to (25.3, 46.2), turned to 0 degrees
- moved R2 14.0 mm to (8.36, 43.6)
- moved R3 14.0 mm to (4.47, 39.5)
- moved GAME 13.8 mm to (8.20, 40.3)
- moved C5 12.3 mm to (25.3, 44.5)
- moved MODE 11.7 mm to (12.6, 41.4)
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Routing:
- net RESET: track 0.00 -> 75.3 mm
- net LD9: track 0.00 -> 57.3 mm
- net LD10: track 0.00 -> 51.5 mm
- net VLIPO: track 0.00 -> 51.1 mm
- net LD11: track 0.00 -> 38.6 mm
- net VCC: track 0.00 -> 31.0 mm, vias 0 -> 3
- net MODE: track 0.00 -> 27.7 mm, vias 0 -> 1
- net RXD: track 0.00 -> 22.4 mm
- net TXD: track 0.00 -> 18.6 mm
- net LD1: track 0.00 -> 16.6 mm
- net LD8: track 0.00 -> 15.3 mm
- net LD2: track 0.00 -> 14.6 mm
- net LD14: track 0.00 -> 13.4 mm
- net LD7: track 0.00 -> 13.3 mm
- net LD5: track 0.00 -> 12.6 mm
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- added copper zone on layer 16, net GND
- added copper zone on layer 1, net VCC

Commit message: small updates after recommendation
Parts:
- moved ON/OFF 2.95 mm to (49.6, 82.0)
- moved LIPO1 2.55 mm to (59.0, 82.4)
Routing:
- net N$7: track 5.03 -> 8.02 mm
- net VLIPO: track 51.1 -> 53.2 mm
Changed lines of the file:
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@@
 <attribute name="VALUE" x="32.766" y="18.5534" size="0.635" layer="28" rot="MR0"/>
 </element>
-<element name="ON/OFF" library="LinnesLab-Switches" package="SWITCH.00" value="SWITCH.JS202011JXQNUPWARDS" x="47.625" y="79.7306" smashed="yes" rot="MR90">
-<attribute name="NAME" x="47.5996" y="75.6666" size="0.6096" layer="26" ratio="20" rot="MR0" align="bottom-center"/>
-<attribute name="VALUE" x="47.625" y="83.6676" size="0.6096" layer="28" ratio="20" rot="MR180" align="top-center"/>
+<element name="ON/OFF" library="LinnesLab-Switches" package="SWITCH.00" value="SWITCH.JS202011JXQNUPWARDS" x="49.5554" y="81.9658" smashed="yes" rot="MR90">
+<attribute name="NAME" x="49.53" y="77.9018" size="0.6096" layer="26" ratio="20" rot="MR0" align="bottom-center"/>
+<attribute name="VALUE" x="49.5554" y="85.9028" size="0.6096" layer="28" ratio="20" rot="MR180" align="top-center"/>
 </element>
 <element name="D4" library="LinnesLab-DiscreteSemi" package="USC" package3d_urn="urn:adsk.eagle:package:15664784/2" value="1A/23V/620mV" x="50.2666" y="72.3138" smashed="yes">
@@
 <attribute name="VALUE" x="56.8198" y="74.1934" size="0.7112" layer="27" rot="R180"/>
 </element>
-<element name="LIPO1" library="LinnesLab-Connectors" package="JST-2-SMD" value="" x="58.1152" y="80.0354" smashed="yes" rot="MR0">
-<attribute name="NAME" x="59.5122" y="81.8134" size="0.6096" layer="26" ratio="20" rot="MR0"/>
-<attribute name="PROD_ID" value="CONN-11443" x="58.1152" y="80.0354" size="1.778" layer="28" rot="MR0" display="off"/>
-<attribute name="SF_ID" value="PRT-08612" x="58.1152" y="80.0354" size="1.778" layer="28" rot="MR0" display="off"/>
-<attribute name="VALUE" x="59.7662" y="80.6704" size="0.6096" layer="28" ratio="20" rot="MR0"/>
+<element name="LIPO1" library="LinnesLab-Connectors" package="JST-2-SMD" value="" x="58.9534" y="82.4484" smashed="yes" rot="MR0">
+<attribute name="NAME" x="60.3504" y="84.2264" size="0.6096" layer="26" ratio="20" rot="MR0"/>
+<attribute name="PROD_ID" value="CONN-11443" x="58.9534" y="82.4484" size="1.778" layer="28" rot="MR0" display="off"/>
+<attribute name="SF_ID" value="PRT-08612" x="58.9534" y="82.4484" size="1.778" layer="28" rot="MR0" display="off"/>
+<attribute name="VALUE" x="60.6044" y="83.0834" size="0.6096" layer="28" ratio="20" rot="MR0"/>
 </element>
 <element name="J1" library="LinnesLab-Connectors" package="2X3-NS" package3d_urn="urn:adsk.eagle:package:18167648/2" value="AVR_SPI_PROG_3X2NS" x="10.541" y="60.4012" smashed="yes">
@@
 <contactref element="U3" pad="3"/>
 <contactref element="C10" pad="1"/>
-<wire x1="57.1152" y1="76.3354" x2="52.6202" y2="76.3354" width="0.1524" layer="16"/>
-<wire x1="52.6202" y1="76.3354" x2="49.2632" y2="79.6924" width="0.1524" layer="16"/>
-<wire x1="49.2632" y1="79.6924" x2="49.225" y2="79.7306" width="0.1524" layer="16"/>
 <wire x1="22.1996" y1="74.4084" x2="19.7643" y2="74.4084" width="0.2032" layer="16"/>
 <wire x1="19.7643" y1="74.4084" x2="19.4412" y2="74.7315" width="0.2032" layer="16"/>
@@
 <wire x1="19.4412" y1="74.7315" x2="19.4412" y2="73.3655125" width="0.2032" layer="16"/>
 <wire x1="19.4412" y1="73.3655125" x2="18.9122" y2="72.8365125" width="0.2032" layer="16"/>
-<wire x1="47.6504" y1="75.9968" x2="47.6504" y2="78.4606" width="0.2032" layer="16"/>
-<wire x1="47.6504" y1="78.4606" x2="48.8822" y2="79.6924" width="0.2032" layer="16"/>
-<wire x1="48.8822" y1="79.6924" x2="49.2632" y2="79.6924" width="0.2032" layer="16"/>
 <wire x1="19.0658875" y1="71.2724" x2="42.926" y2="71.2724" width="0.2032" layer="16"/>
 <wire x1="42.926" y1="71.2724" x2="47.6504" y2="75.9968" width="0.2032" layer="16"/>
+<wire x1="47.6504" y1="75.9968" x2="49.53" y2="77.8764" width="0.1524" layer="16"/>
+<wire x1="49.53" y1="77.8764" x2="49.53" y2="81.026" width="0.1524" layer="16"/>
+<wire x1="49.53" y1="81.026" x2="50.4698" y2="81.9658" width="0.1524" layer="16"/>
+<wire x1="50.4698" y1="81.9658" x2="51.054" y2="81.9658" width="0.1524" layer="16"/>
+<wire x1="51.054" y1="81.9658" x2="51.1554" y2="81.9658" width="0.1524" layer="16"/>
+<wire x1="57.9534" y1="78.7484" x2="54.2714" y2="78.7484" width="0.1524" layer="16"/>
+<wire x1="54.2714" y1="78.7484" x2="51.054" y2="81.9658" width="0.1524" layer="16"/>
 </signal>
 <signal name="N$7">
@@
 <wire x1="49.1166" y1="74.7268" x2="49.149" y2="74.7268" width="0.2032" layer="1"/>
 <via x="49.149" y="74.7268" extent="1-16" drill="0.35"/>
-<wire x1="49.149" y1="74.7268" x2="49.149" y2="77.2306" width="0.2032" layer="16"/>
-<wire x1="49.149" y1="77.2306" x2="49.225" y2="77.2306" width="0.2032" layer="16"/>
+<wire x1="51.1554" y1="79.4658" x2="51.1554" y2="76.7332" width="0.1524" layer="16"/>
+<wire x1="51.1554" y1="76.7332" x2="49.149" y2="74.7268" width="0.1524" layer="16"/>
 </signal>
 <signal name="LD10">

Commit message: updates after 4/3
Parts:
- moved FTDI1 20.2 mm to (31.8, 2.29)
- moved D2 14.6 mm to (31.8, 5.64)
- moved ON/OFF 5.25 mm to (44.8, 79.8)
- moved USB1 2.15 mm to (31.8, 82.8)
- moved C5 2.04 mm to (23.2, 44.4)
- moved C4 2.03 mm to (23.3, 45.8)
- moved XTAL 1.67 mm to (26.4, 45.8)
- moved ACT 1.07 mm to (35.6, 18.8)
- moved RT 0.48 mm to (55.6, 18.8)
- moved LIPO1 0.18 mm to (59.1, 82.5)
- flipped D4 to the bottom, turned to 180 degrees
- turned J1 to 270 degrees
- flipped LED6 to the bottom, turned to 0 degrees
Routing:
- net DTR: track 0.00 -> 31.3 mm
- net TXD: track 18.6 -> 45.1 mm
- net VCC: track 31.0 -> 56.1 mm, vias 3 -> 13
- net RXD: track 22.4 -> 39.6 mm
- net N$16: track 21.5 -> 29.0 mm
- net LD10: track 51.5 -> 46.3 mm
- net N$19: track 25.8 -> 30.1 mm
- net RESET: track 75.3 -> 71.9 mm
- net N$28: track 4.25 -> 6.60 mm
- net LD9: track 57.3 -> 59.6 mm
- net N$20: track 3.83 -> 6.07 mm
- net N$9: track 2.13 -> 4.29 mm
- net GND: track 4.80 -> 6.86 mm
- net N$7: track 8.02 -> 6.16 mm, vias 1 -> 0
- net N$15: track 22.9 -> 21.2 mm
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
Commit message: changes 4/17
Routing:
- net N$19: track 30.1 -> 75.1 mm, vias 2 -> 3
Changed lines of the file:
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@@
 </element>
 <element name="RIGHT" library="LinnesLab-Switches" package="SPST.KT11P4SM34LFS" value="" x="52.07" y="10.414" smashed="yes" rot="R180">
-<attribute name="NAME" x="52.3748" y="8.7122" size="0.762" layer="25" rot="R180"/>
+<attribute name="NAME" x="55.1688" y="9.7028" size="0.762" layer="25" rot="R180"/>
 <attribute name="VALUE" x="57.15" y="14.859" size="0.762" layer="27" rot="R180"/>
 </element>
 <element name="ACTION" library="LinnesLab-Switches" package="SPST.KT11P4SM34LFS" value="" x="31.75" y="10.414" smashed="yes" rot="R180">
+<attribute name="ACTION" value="" x="31.75" y="10.414" size="1.778" layer="27" rot="R180" display="off"/>
 <attribute name="NAME" x="33.5788" y="11.8872" size="0.762" layer="25" rot="R180"/>
 <attribute name="VALUE" x="36.83" y="14.859" size="0.762" layer="27" rot="R180"/>
@@
 <wire x1="47.9298" y1="14.2748" x2="47.9298" y2="15.4804" width="0.1524" layer="16"/>
 <wire x1="47.9298" y1="15.4804" x2="47.9688" y2="15.5194" width="0.1524" layer="16"/>
+<wire x1="56.1975" y1="12.434" x2="58.8264" y2="15.0629" width="0.1524" layer="1"/>
+<wire x1="58.8264" y1="15.0629" x2="58.8264" y2="34.5694" width="0.1524" layer="1"/>
+<wire x1="58.8264" y1="34.5694" x2="51.9684" y2="41.4274" width="0.1524" layer="1"/>
+<wire x1="51.9684" y1="41.4274" x2="39.8272" y2="41.4274" width="0.1524" layer="1"/>
+<via x="39.8272" y="41.4274" extent="1-16" drill="0.35"/>
 </signal>
 <signal name="N$20">
@@
 <contactref element="R24" pad="1"/>
 <contactref element="U1" pad="1"/>
-<wire x1="26.543" y1="38.2718" x2="28.1432" y2="39.872" width="0.1524" layer="16"/>
-<wire x1="26.543" y1="27.3659125" x2="26.543" y2="38.2718" width="0.1524" layer="16"/>
+<wire x1="28.0924" y1="39.8212" x2="28.1432" y2="39.872" width="0.1524" layer="16"/>
+<wire x1="28.0924" y1="28.9153125" x2="28.0924" y2="39.8212" width="0.1524" layer="16"/>
 <wire x1="25.4254" y1="26.709" x2="25.8860875" y2="26.709" width="0.1524" layer="16"/>
-<wire x1="25.8860875" y1="26.709" x2="26.543" y2="27.3659125" width="0.1524" layer="16"/>
+<wire x1="25.8860875" y1="26.709" x2="28.0924" y2="28.9153125" width="0.1524" layer="16"/>
 </signal>
 <signal name="LD7">
