File: Hardware/MakerTherapyBadge.sch (EAGLE design)
At the start: 16 parts, among them J1 AVR_SPI_PROG_3X2NS, U1 ATMEGA328P_TQFP

Commit message: finished schematic
Parts:
- added ACT, EMOJI, GAME, LED6, LED7, LT, RT: (no value), LinnesLab-LED:LED0603
- added ACTION, LEFT, RIGHT: (no value), LinnesLab-Switches:SPST.KT11P4SM34LFS
- added C10, C13, C14, C15: 4.7u, LinnesLab-Passives:CAPACITOR0603
- added C11, C7: (no value), LinnesLab-Passives:CAPACITOR0603
- added C12, C17, C8, C9: 100n, LinnesLab-Passives:CAPACITOR0603
- added C16: 2.2u, LinnesLab-Passives:CAPACITOR0603
- added C18: 1u, LinnesLab-Passives:CAPACITOR0603
- added D1: 1A/23V/620mV, LinnesLab-DiscreteSemi:SCHOTTKY-USC
- added LED8: (no value), adafruit:SEGMENT_8X8_ROWCATHODEM12A881UR
- added MODE: SWITCH.JS202011JXQNUPWARDS, LinnesLab-Switches:SWITCH.JS202011JXQNUPWARDS
- added OP1: (no value), LinnesLab-AnalogIC:OP-SINGLEOT
- added R10, R2, R3, R5: 1k, LinnesLab-Passives:RESISTOR0603
- added R11, R17, R4, R7, R8: 10k, LinnesLab-Passives:RESISTOR0603
- added R12: 487, LinnesLab-Passives:RESISTOR0603
- added R13: 12k, LinnesLab-Passives:RESISTOR0603
- added R14, R15: 210k, LinnesLab-Passives:RESISTOR0603
- added R16: 3.3M, LinnesLab-Passives:RESISTOR0603
- added R18, R19, R20, R21, R22, R23, R24, R25: 205, LinnesLab-Passives:RESISTOR0603
- added R6, R9: (no value), LinnesLab-Passives:RESISTOR0603
- added U$1: ADPS9008, LinnesLab-Sensors:ADPS9008
- added U3: MCP73831.SOT23-5, LinnesLab-Power:MCP73831.SOT23-5
- added USB1: USB.MICRO.PWR-BIGGERPADS, LinnesLab-Connectors:USB.MICRO.PWR-BIGGERPADS
Connections:
- new net ACTION: U1.ADC6
- new net LD1: R22.1, U1.D4/PD4(XCK/T0)
- new net LD10: J1.1, LED8.A4, U1.D12/PB4(MISO)
- new net LD11: J1.4, LED8.A6, U1.D11/PB3(MOSI/OC2)
- new net LD12: R21.1, U1.D10/PB2(SS/OC1B)
- new net LD13: LED8.A1, U1.D9/PB1(OC1A)
- new net LD14: R19.1, U1.D8/PB0(ICP)
- new net LD15: LED8.A7, U1.D7/PD7(AIN1)
- new net LD16: LED8.A8, U1.D6/PD6(AIN0)
- new net LD2: R24.1, U1.D3/PD3(INT1)
- new net LD3: LED8.A2, U1.D2/PD2(INT0)
- new net LD4: LED8.A3, U1.PC5(ADC5/SCL)
- new net LD5: R25.1, U1.PC4(ADC4/SDA)
- new net LD6: LED8.A5, U1.PC3(ADC3)
- new net LD7: R23.1, U1.PC2(ADC2)
- new net LD8: R20.1, U1.PC1(ADC1)
- new net LD9: J1.3, R18.1, U1.D13/PB5(SCK)
- new net LEFT: U1.PC0(ADC0)
- new net MODE: GAME.A, MODE.2, R2.1, U1.D5/PD5(T1)
- new net N$10: LT.C, R9.2
- new net N$14: GAME.C, R3.2
- new net N$15: C9.1, LEFT.B, LT.A, R8.2
- new net N$16: ACT.A, ACTION.B, C7.2, R4.2
- new net N$17: ACT.C, R5.2
- new net N$18: R6.2, RT.C
- new net N$19: C8.2, R7.2, RIGHT.B, RT.A
- new net N$20: D1.A, USB1.V+
- new net N$21: LED6.A, R10.1
- new net N$22: LED8.K8, R25.2
- new net N$23: LED7.C, R12.2
- new net N$24: R11.2, U3.PROG
- new net N$25: OP1G$1.-IN, R16.2, R17.1
- new net N$27: C16.2, OP1G$1.+IN, R14.1, R15.2
- new net N$28: C13.2, R13.2, U$1.OUT
- new net N$30: C13.1, C14.1, C15.1
- new net N$31: C15.2, C16.1, R17.2
- new net N$8: EMOJI.C, R2.2
- new net PULSE: OP1G$1.OUT, R16.1
- new net RIGHT: U1.ADC7
- new net RXD: FTDI1.CTS, U1.D0/PD0(RXD)
- new net STAT: LED6.C, U3.STAT
- new net TXD: FTDI1.VCC, U1.D1/PD1(TXD)
- net DTR: now also FTDI1.GND
- net GND: now also C10.2, C11.2, C12.1, C14.2, C17.2, C18.2, C7.1, C8.1, C9.2, FTDI1.DTR, FTDI1.RXI, MODE.1, OP1G$2.V-, R11.1, R12.1, R13.1, R15.1, R3.1, R4.1, R5.1, R6.1, R7.1, R8.1, R9.1, U$1.GND, U3.VSS, USB1.GND
- net N$1: now also LED8.K1, R18.2; no longer FTDI1.DTR, FTDI1.RXI
- net N$11: now also LED8.K5, R22.2; no longer J1.1
- net N$12: now also LED8.K6, R23.2; no longer J1.3
- net N$13: now also LED8.K7, R24.2; no longer J1.5
- net N$3: now also LED8.K2, R19.2; no longer FTDI1.VCC
- net N$4: now also LED8.K3, R20.2; no longer FTDI1.CTS
- net N$5: now also LED8.K4, R21.2; no longer FTDI1.GND
- net RESET: now also J1.5
- net VCC: now also ACTION.A, C11.1, C12.2, C17.1, C18.1, D1.C, EMOJI.A, LED7.A, LEFT.A, MODE.3, OP1G$2.V+, R10.2, R14.2, RIGHT.A, U$1.VCC, U3.VIN
- net VLIPO: now also C10.1, U3.VBAT
Other:
- note added: "Action Buttons"
- note added: "Sihun Kim Therapy Mood Badge 1.0"

Commit message: updates from 3/20
Parts:
- C7: value (none) -> 100n
- R6, R9: value (none) -> 1k
Changed lines of the file:
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@@
 <part name="R4" library="LinnesLab-Passives" deviceset="RESISTOR" device="0603" package3d_urn="urn:adsk.eagle:package:15661944/2" value="10k"/>
 <part name="R5" library="LinnesLab-Passives" deviceset="RESISTOR" device="0603" package3d_urn="urn:adsk.eagle:package:15661944/2" value="1k"/>
-<part name="R6" library="LinnesLab-Passives" deviceset="RESISTOR" device="0603" package3d_urn="urn:adsk.eagle:package:15661944/2"/>
+<part name="R6" library="LinnesLab-Passives" deviceset="RESISTOR" device="0603" package3d_urn="urn:adsk.eagle:package:15661944/2" value="1k"/>
 <part name="R7" library="LinnesLab-Passives" deviceset="RESISTOR" device="0603" package3d_urn="urn:adsk.eagle:package:15661944/2" value="10k"/>
-<part name="C7" library="LinnesLab-Passives" deviceset="CAPACITOR" device="0603" package3d_urn="urn:adsk.eagle:package:15661989/2"/>
+<part name="C7" library="LinnesLab-Passives" deviceset="CAPACITOR" device="0603" package3d_urn="urn:adsk.eagle:package:15661989/2" value="100n"/>
 <part name="C8" library="LinnesLab-Passives" deviceset="CAPACITOR" device="0603" package3d_urn="urn:adsk.eagle:package:15661989/2" value="100n"/>
 <part name="GND12" library="LinnesLab-Symbols" deviceset="GND" device=""/>
@@
 <part name="C9" library="LinnesLab-Passives" deviceset="CAPACITOR" device="0603" package3d_urn="urn:adsk.eagle:package:15661989/2" value="100n"/>
 <part name="R8" library="LinnesLab-Passives" deviceset="RESISTOR" device="0603" package3d_urn="urn:adsk.eagle:package:15661944/2" value="10k"/>
-<part name="R9" library="LinnesLab-Passives" deviceset="RESISTOR" device="0603" package3d_urn="urn:adsk.eagle:package:15661944/2"/>
+<part name="R9" library="LinnesLab-Passives" deviceset="RESISTOR" device="0603" package3d_urn="urn:adsk.eagle:package:15661944/2" value="1k"/>
 <part name="GND18" library="LinnesLab-Symbols" deviceset="GND" device=""/>
 <part name="GND19" library="LinnesLab-Symbols" deviceset="GND" device=""/>
